File: ProbeStationBreakoutBox/carrier_breakout_box_make-before-break.sch (EAGLE design)
At the start: 77 parts, among them X1 A1944-50, X10 A1944-50, X11 A1944-50, X12 A1944-50, X13 A1944-50, X14 A1944-50, X15 A1944-50, X16 A1944-50, X17 A1944-50, X18 A1944-50, X19 A1944-50, X2 A1944-50, X20 A1944-50, X21 A1944-50, X22 A1944-50, X23 A1944-50, X24 A1944-50, X25 A1944-50, X3 A1944-50, X4 A1944-50, X5 A1944-50, X6 A1944-50, X7 A1944-50, X8 A1944-50, X9 A1944-50

Commit message: Updated
Connections:
- removed net N$8: S1.S, S10.S, S11.S, S12.S, S13.S, S14.S, S15.S, S16.S, S17.S, S18.S, S19.S, S2.S, S20.S, S21.S, S22.S, S23.S, S24.S, S25.S, S26.S, S27.S, S28.S, S29.S, S3.S, S30.S, S31.S, S32.S, S33.S, S34.S, S35.S, S36.S, S37.S, S38.S, S39.S, S4.S, S40.S, S41.S, S42.S, S43.S, S44.S, S45.S, S46.S, S47.S, S48.S, S5.S, S6.S, S7.S, S8.S, S9.S, X25.1, X25.2
- new net N$7: S1.S, S10.S, S11.S, S12.S, S13.S, S14.S, S15.S, S16.S, S17.S, S18.S, S19.S, S2.S, S20.S, S21.S, S22.S, S23.S, S24.S, S25.S, S26.S, S27.S, S28.S, S29.S, S3.S, S30.S, S31.S, S32.S, S33.S, S34.S, S35.S, S36.S, S37.S, S38.S, S39.S, S4.S, S40.S, S41.S, S42.S, S43.S, S44.S, S45.S, S46.S, S47.S, S48.S, S5.S, S6.S, S7.S, S8.S, S9.S, X1.2, X10.2, X11.2, X12.2, X13.2, X14.2, X15.2, X16.2, X17.2, X18.2, X19.2, X2.2, X20.2, X21.2, X22.2, X23.2, X24.2, X25.2, X3.2, X4.2, X5.2, X6.2, X7.2, X8.2, X9.2
Other:
- moved on the sheet: X25

Commit message: Added banana connectors to breakout box circuit
Parts:
- added J1, J10, J11, J12, J13, J14, J15, J16, J17, J18, J19, J2, J20, J21, J22, J23, J24, J3, J4, J5, J6, J7, J8, J9: (no value), SparkFun-Connectors:BANANA_CONN
Connections:
- net N$21: now also J24.1
- net N$22: now also J23.1
- net N$23: now also J22.1
- net N$24: now also J21.1
- net N$25: now also J20.1
- net N$33: now also J19.1
- net N$46: now also J18.1
- net N$49: now also J2.1
- net N$50: now also J3.1
- net N$51: now also J4.1
- net N$52: now also J17.1
- net N$53: now also J5.1
- net N$54: now also J6.1
- net N$55: now also J16.1
- net N$58: now also J15.1
- net N$61: now also J14.1
- net N$64: now also J13.1
- net N$66: now also J7.1
- net N$67: now also J8.1
- net N$68: now also J9.1
- net N$69: now also J10.1
- net N$70: now also J11.1
- net N$71: now also J12.1
